File: espled/espled.kicad_pcb (KiCad board)
At the start: 2 copper layers, 60 x 44 mm, 34 parts, among them J1 Screw_Terminal_01x02, J2 Barrel_Jack_Switch, J3 Screw_Terminal_01x03, J4 Screw_Terminal_01x03, J5 Screw_Terminal_01x03, J6 Screw_Terminal_01x03, J7 Conn_01x03, SW1 SW_Push, SW2 SW_Push, U1 AP2112K-3.3, U2 ESP32-WROOM-32, U3 74HCT245

Commit message: Prepare Rev1.
Parts:
- removed J6: Screw_Terminal_01x03, TerminalBlock_Phoenix:TerminalBlock_Phoenix_PT-1,5-3-5.0-H_1x03_P5.00mm_Horizontal
- removed R9: 330, Resistor_SMD:R_0603_1608Metric
- moved J5 15.8 mm to (81.0, 90.2)
- moved J3 11.9 mm to (99.0, 73.0)
- moved J4 11.7 mm to (99.0, 90.0)
- moved C4 4.50 mm to (86.0, 63.0)
- moved C6 4.50 mm to (88.0, 63.0)
- moved C8 4.50 mm to (90.0, 63.0)
- moved R6 4.10 mm to (89.4, 68.5)
- moved R8 3.90 mm to (89.4, 72.5)
- moved R7 0.10 mm to (89.4, 70.5)
Connections:
- R6 pad 2: /CH3 -> /CH1
- R8 pad 2: /CH1 -> /CH3
- U2 pad 31: /IO19 -> Net-(U2-Pad31)
- U3 pad 15: /CH4 -> Net-(U3-Pad15)
- U3 pad 5: /IO19 -> GND
Routing:
- net Net-(J3-Pad2): track 73.5 -> 9.03 mm, vias 0 -> 1
- net Net-(J4-Pad2): track 56.4 -> 26.3 mm, vias 0 -> 1
- net Net-(J6-Pad2): track 26.4 -> 0.00 mm
- net /IO19: track 23.4 -> 0.00 mm, vias 2 -> 0
- net GND: track 62.1 -> 83.3 mm
- net Net-(J5-Pad2): track 33.7 -> 19.4 mm
- net /CH4: track 5.08 -> 0.00 mm
Other:
- board size 60 x 44 mm -> 51.5 x 44 mm
- board text added: "+"
- board text added: "-"
- board text added: "CH1"
- board text added: "CH2"
- board text added: "CH3"
- board text added: "D"
- board text added: "ESPLED"
- board text added: "FLASH"
- board text added: "GND"
- board text added: "POWER"
- board text added: "RESET"
- board text added: "RX"
- board text added: "Rev 1 (C) 2020 Matir 5V Only"
- board text added: "TX"
- board text added: "UART"
