File: pcbs/ornament2020/ornament/ornament.kicad_pcb (KiCad board)
At the start: 2 copper layers, 55 x 96 mm, 28 parts, among them J1 PROG, U1 ATtiny84-20SSU, U2 TPS61099X, U3 AT42QT1010-TSHR

Commit message: Update tapeout
Routing:
- net /PB1: track 17.8 -> 13.6 mm
- net /PB0: track 39.6 -> 35.9 mm
Changed lines of the file:
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@@
     (thickness 1.6)
     (drawings 20)
-    (tracks 178)
+    (tracks 177)
     (zones 0)
     (modules 28)
@@
       (plotinvisibletext false)
       (padsonsilk false)
-      (subtractmaskfromsilk false)
+      (subtractmaskfromsilk true)
       (outputformat 1)
       (mirror false)
-      (drillshape 1)
+      (drillshape 0)
       (scaleselection 1)
-      (outputdirectory ""))
+      (outputdirectory "output/"))
   )
   (net 0 "")
@@
   (segment (start 160 92.8) (end 160.2 93) (width 0.254) (layer B.Cu) (net 16))
   (segment (start 160 90.775) (end 160 92.8) (width 0.254) (layer B.Cu) (net 16))
-  (segment (start 168.25 62.325) (end 167.175 62.325) (width 0.254) (layer B.Cu) (net 17))
-  (segment (start 167.175 62.325) (end 165.25 64.25) (width 0.254) (layer B.Cu) (net 17))
-  (segment (start 165.25 64.25) (end 165.25 72.5) (width 0.254) (layer B.Cu) (net 17))
-  (segment (start 165.62 72.87) (end 170.85 72.87) (width 0.254) (layer B.Cu) (net 17))
-  (segment (start 165.25 72.5) (end 165.62 72.87) (width 0.254) (layer B.Cu) (net 17))
-  (segment (start 170.85 74.14) (end 166.14 74.14) (width 0.254) (layer B.Cu) (net 18))
-  (segment (start 166.14 74.14) (end 164.75 72.75) (width 0.254) (layer B.Cu) (net 18))
-  (segment (start 164.75 72.75) (end 164.75 59.75) (width 0.254) (layer B.Cu) (net 18))
-  (segment (start 164.75 59.75) (end 167.75 56.75) (width 0.254) (layer B.Cu) (net 18))
+  (segment (start 168.25 62.325) (end 167 63.575) (width 0.254) (layer B.Cu) (net 17))
+  (segment (start 169.294038 72.87) (end 170.85 72.87) (width 0.254) (layer B.Cu) (net 17))
+  (segment (start 167 70.575962) (end 169.294038 72.87) (width 0.254) (layer B.Cu) (net 17))
+  (segment (start 167 63.575) (end 167 70.575962) (width 0.254) (layer B.Cu) (net 17))
   (segment (start 167.75 56.75) (end 176.25 56.75) (width 0.254) (layer B.Cu) (net 18))
   (segment (start 178.69799 61.77299) (end 179.5 62.575) (width 0.254) (layer B.Cu) (net 18))
   (segment (start 178.69799 59.19799) (end 178.69799 61.77299) (width 0.254) (layer B.Cu) (net 18))
   (segment (start 176.25 56.75) (end 178.69799 59.19799) (width 0.254) (layer B.Cu) (net 18))
+  (segment (start 169.921971 74.14) (end 170.85 74.14) (width 0.254) (layer B.Cu) (net 18))
+  (segment (start 166.54599 70.764019) (end 169.921971 74.14) (width 0.254) (layer B.Cu) (net 18))
+  (segment (start 166.54599 57.95401) (end 166.54599 70.764019) (width 0.254) (layer B.Cu) (net 18))
+  (segment (start 167.75 56.75) (end 166.54599 57.95401) (width 0.254) (layer B.Cu) (net 18))
   (segment (start 180.495 70.33) (end 180.5 70.325) (width 0.254) (layer B.Cu) (net 19))
   (segment (start 175.8 70.33) (end 180.495 70.33) (width 0.254) (layer B.Cu) (net 19))

Commit message: Ornament bump
Parts:
- added JP1: Jumper_NO_Small, Jumper:SolderJumper-2_P1.3mm_Open_TrianglePad1.0x1.5mm, B.Cu at (154.5, 89.8)
- added REF**: MountingHole_3.5mm, MountingHole:MountingHole_3.5mm, F.Cu at (173.2, 29.8)
Routing:
- net VCC: track 95.5 -> 102.3 mm
- net GND: track 36.5 -> 39.7 mm
- net Net-(BT1-Pad1): track 19.4 -> 22.2 mm
Other:
- board text added: "2020"
- board text added: "Happy Holidays! - David & Ann"
Changed lines of the file:
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@@
   (general
     (thickness 1.6)
-    (drawings 20)
-    (tracks 177)
+    (drawings 24)
+    (tracks 183)
     (zones 0)
-    (modules 28)
+    (modules 30)
     (nets 26)
   )
@@
   )
   (setup
-    (last_trace_width 0.254)
+    (last_trace_width 0.5)
     (user_trace_width 0.254)
     (user_trace_width 0.5)
@@
     (add_net VCC)
   )
+  (module MountingHole:MountingHole_3.5mm (layer F.Cu)
+    (at 173.25 29.75)
+    (descr "Mounting Hole 3.5mm, no annular")
+    (tags "mounting hole 3.5mm no annular")
+    (attr virtual)
+    (fp_text reference REF** (at 0 -4.5) (layer F.SilkS)
+      (effects (font (size 1 1) (thickness 0.15)))
+    )
+    (fp_text value MountingHole_3.5mm (at 0 4.5) (layer F.Fab)
+      (effects (font (size 1 1) (thickness 0.15)))
+    )
+    (fp_text user %R (at 0.3 0) (layer F.Fab)
+      (effects (font (size 1 1) (thickness 0.15)))
+    )
+    (fp_circle (center 0 0) (end 3.5 0) (layer Cmts.User) (width 0.15))
+    (fp_circle (center 0 0) (end 3.75 0) (layer F.CrtYd) (width 0.05))
+    (pad 1 np_thru_hole circle (at 0 0) (size 3.5 3.5) (drill 3.5) (layers *.Cu *.Mask))
+  )
   (module Battery:BatteryHolder_Keystone_3002_1x2032 (layer B.Cu)
     (at 173.4 98)
     (descr https://www.tme.eu/it/Document/a823211ec201a9e209042d155fe22d2b/KEYS2996.pdf)
     (tags "BR2016 CR2016 DL2016 BR2020 CL2020 BR2025 CR2025 DL2025 DR2032 CR2032 DL2032")
+    (zone_connect 2)
     (attr smd)
     (fp_text reference BT1 (at -9.15 -9.7) (layer B.SilkS)
@@
     (fp_arc (start 0 0) (end 3.9 9.8) (angle 43.40107348) (layer B.CrtYd) (width 0.05))
     (fp_arc (start 0 0) (end 3.85 9.5) (angle 44.1) (layer B.SilkS) (width 0.12))
-    (pad "" smd rect (at 12.8 0) (size 5.1 5.1) (layers B.Cu B.Paste B.Mask))
+    (pad "" smd rect (at 12.8 0) (size 5.1 5.1) (layers B.Cu B.Paste B.Mask)
+      (zone_connect 2))
     (pad 1 smd rect (at -12.8 0) (size 5.1 5.1) (layers B.Cu B.Paste B.Mask)
-      (net 1 "Net-(BT1-Pad1)"))
+      (net 1 "Net-(BT1-Pad1)") (zone_connect 2))
     (pad 2 smd circle (at 0 0) (size 17.8 17.8) (layers B.Cu B.Mask)
-      (net 2 GND))
+      (net 2 GND) (zone_connect 2))
     (model ${KISYS3DMOD}/Battery.3dshapes/BatteryHolder_Keystone_3002_1x2032.wrl
       (at (xyz 0 0 0))
@@
     )
   )
+  (module Jumper:SolderJumper-2_P1.3mm_Open_TrianglePad1.0x1.5mm (layer B.Cu)
+    (at 154.5 89.75 270)
+    (descr "SMD Solder Jumper, 1x1.5mm Triangular Pads, 0.3mm gap, open")
+    (tags "solder jumper open")
+    (attr virtual)
+    (fp_text reference JP1 (at 0 1.8 270) (layer B.SilkS)
+      (effects (font (size 1 1) (thickness 0.15)) (justify mirror))
+    )
+    (fp_text value Jumper_NO_Small (at 0 -1.9 270) (layer B.Fab)
+      (effects (font (size 1 1) (thickness 0.15)) (justify mirror))
+    )
+    (fp_line (start 1.65 -1.25) (end -1.65 -1.25) (layer B.CrtYd) (width 0.05))
+    (fp_line (start 1.65 -1.25) (end 1.65 1.25) (layer B.CrtYd) (width 0.05))
+    (fp_line (start -1.65 1.25) (end -1.65 -1.25) (layer B.CrtYd) (width 0.05))
+    (fp_line (start -1.65 1.25) (end 1.65 1.25) (layer B.CrtYd) (width 0.05))
+    (fp_line (start -1.4 1) (end 1.4 1) (layer B.SilkS) (width 0.12))
+    (fp_line (start 1.4 1) (end 1.4 -1) (layer B.SilkS) (width 0.12))
+    (fp_line (start 1.4 -1) (end -1.4 -1) (layer B.SilkS) (width 0.12))
+    (fp_line (start -1.4 -1) (end -1.4 1) (layer B.SilkS) (width 0.12))
+    (pad 2 smd custom (at 0.725 0 270) (size 0.3 0.3) (layers B.Cu B.Mask)
+      (net 1 "Net-(BT1-Pad1)") (zone_connect 2)
+      (options (clearance outline) (anchor rect))
+      (primitives
+        (gr_poly (pts
+           (xy -0.65 0.75) (xy 0.5 0.75) (xy 0.5 -0.75) (xy -0.65 -0.75) (xy -0.15 0)
+) (width 0))
+      ))
+    (pad 1 smd custom (at -0.725 0 270) (size 0.3 0.3) (layers B.Cu B.Mask)
+      (net 3 VCC) (zone_connect 2)
+      (options (clearance outline) (anchor rect))
+      (primitives
+        (gr_poly (pts
+           (xy -0.5 0.75) (xy 0.5 0.75) (xy 1 0) (xy 0.5 -0.75) (xy -0.5 -0.75)
+) (width 0))
+      ))
+  )
+  (dimension 54.75 (width 0.15) (layer Dwgs.User)
+    (gr_text "54.750 mm" (at 173.375 124.3) (layer Dwgs.User)
+      (effects (font (size 1 1) (thickness 0.15)))
+    )
+    (feature1 (pts (xy 146 120) (xy 146 123.586421)))
+    (feature2 (pts (xy 200.75 120) (xy 200.75 123.586421)))
+    (crossbar (pts (xy 200.75 123) (xy 146 123)))
+    (arrow1a (pts (xy 146 123) (xy 147.126504 122.413579)))
+    (arrow1b (pts (xy 146 123) (xy 147.126504 123.586421)))
+    (arrow2a (pts (xy 200.75 123) (xy 199.623496 122.413579)))
+    (arrow2b (pts (xy 200.75 123) (xy 199.623496 123.586421)))
+  )
+  (dimension 96 (width 0.15) (layer Dwgs.User)
+    (gr_text "96.000 mm" (at 208.55 72 90) (layer Dwgs.User)
+      (effects (font (size 1 1) (thickness 0.15)))
+    )
+    (feature1 (pts (xy 205 24) (xy 207.836421 24)))
+    (feature2 (pts (xy 205 120) (xy 207.836421 120)))
+    (crossbar (pts (xy 207.25 120) (xy 207.25 24)))
+    (arrow1a (pts (xy 207.25 24) (xy 207.836421 25.126504)))
+    (arrow1b (pts (xy 207.25 24) (xy 206.663579 25.126504)))
+    (arrow2a (pts (xy 207.25 120) (xy 207.836421 118.873496)))
+    (arrow2b (pts (xy 207.25 120) (xy 206.663579 118.873496)))
+  )
+  (gr_text "Happy\nHolidays!\n\n- David & Ann" (at 173.5 48.5) (layer B.SilkS)
+    (effects (font (size 2 2) (thickness 0.3)) (justify mirror))
+  )
+  (gr_text 2020 (at 172.25 114) (layer B.SilkS)
+    (effects (font (size 7.5 7.5) (thickness 1.3) italic) (justify mirror))
+  )
   (gr_line (start 159.5 120) (end 187 120) (layer Edge.Cuts) (width 0.05))
   (gr_line (start 145.75 96.25) (end 159.5 120) (layer Edge.Cuts) (width 0.05))
@@
   (segment (start 160.6 95.15) (end 160.6 98) (width 0.254) (layer B.Cu) (net 1))
   (segment (start 161.5 94.25) (end 160.6 95.15) (width 0.254) (layer B.Cu) (net 1))
+  (segment (start 154.7625 90.7375) (end 154.5 90.475) (width 0.5) (layer B.Cu) (net 1))
+  (segment (start 157.2 90.7375) (end 154.7625 90.7375) (width 0.5) (layer B.Cu) (net 1))
   (segment (start 159.35 89.15) (end 160 89.8) (width 0.254) (layer B.Cu) (net 2))
   (segment (start 159.35 88.825) (end 159.35 89.15) (width 0.254) (layer B.Cu) (net 2))
@@
   (via (at 171 58.75) (size 0.8) (drill 0.4) (layers F.Cu B.Cu) (net 2))
   (segment (start 171 60.4) (end 171 58.75) (width 0.254) (layer B.Cu) (net 2))
+  (segment (start 158.1375 89.8) (end 157.2 88.8625) (width 0.5) (layer B.Cu) (net 2))
+  (segment (start 160 89.8) (end 158.1375 89.8) (width 0.5) (layer B.Cu) (net 2))
   (segment (start 160 88.825) (end 160 88.5) (width 0.254) (layer B.Cu) (net 3))
   (segment (start 160 87.4625) (end 160.4625 87) (width 0.5) (layer B.Cu) (net 3))
@@
   (segment (start 173 70.5) (end 173 66.175) (width 0.254) (layer B.Cu) (net 3))
   (segment (start 173 74.235) (end 173 70.5) (width 0.254) (layer B.Cu) (net 3))
+  (segment (start 156.525 87) (end 160.4625 87) (width 0.5) (layer B.Cu) (net 3))
+  (segment (start 154.5 89.025) (end 156.525 87) (width 0.5) (layer B.Cu) (net 3))
   (segment (start 188.4 104.45) (end 188.5 104.35) (width 0.254) (layer B.Cu) (net 4))
   (segment (start 188.4 106.2) (end 188.4 104.45) (width 0.254) (layer B.Cu) (net 4))
