File: pcbs/ornament2020/ornament/ornament.sch (KiCad schematic (older format))
At the start: 22 parts, among them J1 PROG, U1 ATtiny84-20SSU, U2 TPS61099X

Commit message: Update ornament
Parts:
- added C5: 10n, Capacitor_SMD:C_0603_1608Metric, symbol Device:C_Small
- added R8: 10k, Resistor_SMD:R_0603_1608Metric, symbol Device:R_Small
- added TP1: Touch, symbol Connector:TestPoint
- added U3: AT42QT1010-TSHR, Package_TO_SOT_SMD:SOT-23-6, symbol Sensor_Touch:AT42QT1010-TSHR
- BT1: footprint (none) -> Battery:BatteryHolder_Keystone_3002_1x2032
- C1: footprint (none) -> Capacitor_SMD:C_0603_1608Metric
- C2, C3, C4: footprint (none) -> Capacitor_SMD:C_0805_2012Metric
- D1, D2, D3, D4, D5, D6: footprint (none) -> LED_SMD:LED_0603_1608Metric
- L1: footprint (none) -> Inductor_SMD:L_1008_2520Metric
- R1, R2, R3, R4, R5, R6, R7: footprint (none) -> Resistor_SMD:R_0603_1608Metric
Connections:
- net GND: now also U3.2 (VSS), U3.6 (SYNC)
- net MISO: now also J1.1 (Pin_1); no longer J1.2 (Pin_2)
- net VCC: now also J1.2 (Pin_2), U3.5 (VDD); no longer J1.1 (Pin_1)
- net PB2: now reaches U1.5 (PB2)
- net PB2: now also U3.1 (OUT)
- new net: C5.1, R8.2, U3.3 (SNSK)
- new net: C5.2, U3.4 (SNS)
- new net: R8.1, TP1.1
- no-connect marks 2 -> 1
Changed lines of the file:
@@
 F 0 "BT1" H 1650 2000 50  0000 L CNN
 F 1 "CR2032" H 1550 1800 50  0000 L CNN
-F 2 "" V 1900 1910 50  0001 C CNN
+F 2 "Battery:BatteryHolder_Keystone_3002_1x2032" V 1900 1910 50  0001 C CNN
 F 3 "~" V 1900 1910 50  0001 C CNN
 	1    1900 1850
@@
 F 0 "L1" V 2290 1550 50  0000 C CNN
 F 1 "2.2uH" V 2199 1550 50  0000 C CNN
-F 2 "" H 2100 1550 50  0001 C CNN
+F 2 "Inductor_SMD:L_1008_2520Metric" H 2100 1550 50  0001 C CNN
 F 3 "~" H 2100 1550 50  0001 C CNN
 	1    2100 1550
@@
 F 0 "C2" H 2242 1846 50  0000 L CNN
 F 1 "10u" H 2242 1755 50  0000 L CNN
-F 2 "" H 2150 1800 50  0001 C CNN
+F 2 "Capacitor_SMD:C_0805_2012Metric" H 2150 1800 50  0001 C CNN
 F 3 "~" H 2150 1800 50  0001 C CNN
 	1    2150 1800
@@
 F 0 "C3" H 3542 1696 50  0000 L CNN
 F 1 "10u" H 3542 1605 50  0000 L CNN
-F 2 "" H 3450 1650 50  0001 C CNN
+F 2 "Capacitor_SMD:C_0805_2012Metric" H 3450 1650 50  0001 C CNN
 F 3 "~" H 3450 1650 50  0001 C CNN
 	1    3450 1650
@@
 F 0 "C4" H 3792 1696 50  0000 L CNN
 F 1 "10u" H 3792 1605 50  0000 L CNN
-F 2 "" H 3700 1650 50  0001 C CNN
+F 2 "Capacitor_SMD:C_0805_2012Metric" H 3700 1650 50  0001 C CNN
 F 3 "~" H 3700 1650 50  0001 C CNN
 	1    3700 1650
@@
 F 0 "C1" H 1142 2996 50  0000 L CNN
 F 1 "C_Small" H 1142 2905 50  0000 L CNN
-F 2 "" H 1050 2950 50  0001 C CNN
+F 2 "Capacitor_SMD:C_0603_1608Metric" H 1050 2950 50  0001 C CNN
 F 3 "~" H 1050 2950 50  0001 C CNN
 	1    1050 2950
@@
 Wire Wire Line
 	3250 4050 2950 4050
-NoConn ~ 2950 3750
-NoConn ~ 2950 4150
 $Comp
 L Device:LED D1
@@
 F 0 "D1" V 4439 3432 50  0000 R CNN
 F 1 "LED" V 4348 3432 50  0000 R CNN
-F 2 "" H 4400 3550 50  0001 C CNN
+F 2 "LED_SMD:LED_0603_1608Metric" H 4400 3550 50  0001 C CNN
 F 3 "~" H 4400 3550 50  0001 C CNN
 	1    4400 3550
@@
 F 0 "D2" V 4689 3432 50  0000 R CNN
 F 1 "LED" V 4598 3432 50  0000 R CNN
-F 2 "" H 4650 3550 50  0001 C CNN
+F 2 "LED_SMD:LED_0603_1608Metric" H 4650 3550 50  0001 C CNN
 F 3 "~" H 4650 3550 50  0001 C CNN
 	1    4650 3550
@@
 F 0 "D3" V 4939 3432 50  0000 R CNN
 F 1 "LED" V 4848 3432 50  0000 R CNN
-F 2 "" H 4900 3550 50  0001 C CNN
+F 2 "LED_SMD:LED_0603_1608Metric" H 4900 3550 50  0001 C CNN
 F 3 "~" H 4900 3550 50  0001 C CNN
 	1    4900 3550
@@
 F 0 "D4" V 5189 3432 50  0000 R CNN
 F 1 "LED" V 5098 3432 50  0000 R CNN
-F 2 "" H 5150 3550 50  0001 C CNN
+F 2 "LED_SMD:LED_0603_1608Metric" H 5150 3550 50  0001 C CNN
 F 3 "~" H 5150 3550 50  0001 C CNN
 	1    5150 3550
@@
 F 0 "D5" V 5439 3432 50  0000 R CNN
 F 1 "LED" V 5348 3432 50  0000 R CNN
-F 2 "" H 5400 3550 50  0001 C CNN
+F 2 "LED_SMD:LED_0603_1608Metric" H 5400 3550 50  0001 C CNN
 F 3 "~" H 5400 3550 50  0001 C CNN
 	1    5400 3550
@@
 F 0 "D6" V 5689 3432 50  0000 R CNN
 F 1 "LED" V 5598 3432 50  0000 R CNN
-F 2 "" H 5650 3550 50  0001 C CNN
+F 2 "LED_SMD:LED_0603_1608Metric" H 5650 3550 50  0001 C CNN
 F 3 "~" H 5650 3550 50  0001 C CNN
 	1    5650 3550
@@
 F 0 "R2" H 4459 3196 50  0000 L CNN
 F 1 "R_Small" H 4459 3105 50  0000 L CNN
-F 2 "" H 4400 3150 50  0001 C CNN
+F 2 "Resistor_SMD:R_0603_1608Metric" H 4400 3150 50  0001 C CNN
 F 3 "~" H 4400 3150 50  0001 C CNN
 	1    4400 3150
@@
 F 0 "R3" H 4709 3196 50  0000 L CNN
 F 1 "R_Small" H 4709 3105 50  0000 L CNN
-F 2 "" H 4650 3150 50  0001 C CNN
+F 2 "Resistor_SMD:R_0603_1608Metric" H 4650 3150 50  0001 C CNN
 F 3 "~" H 4650 3150 50  0001 C CNN
 	1    4650 3150
@@
 F 0 "R4" H 4959 3196 50  0000 L CNN
 F 1 "R_Small" H 4959 3105 50  0000 L CNN
-F 2 "" H 4900 3150 50  0001 C CNN
+F 2 "Resistor_SMD:R_0603_1608Metric" H 4900 3150 50  0001 C CNN
 F 3 "~" H 4900 3150 50  0001 C CNN
 	1    4900 3150
@@
 F 0 "R5" H 5209 3196 50  0000 L CNN
 F 1 "R_Small" H 5209 3105 50  0000 L CNN
-F 2 "" H 5150 3150 50  0001 C CNN
+F 2 "Resistor_SMD:R_0603_1608Metric" H 5150 3150 50  0001 C CNN
 F 3 "~" H 5150 3150 50  0001 C CNN
 	1    5150 3150
@@
 F 0 "R6" H 5459 3196 50  0000 L CNN
 F 1 "R_Small" H 5459 3105 50  0000 L CNN
-F 2 "" H 5400 3150 50  0001 C CNN
+F 2 "Resistor_SMD:R_0603_1608Metric" H 5400 3150 50  0001 C CNN
 F 3 "~" H 5400 3150 50  0001 C CNN
 	1    5400 3150
@@
 F 0 "R7" H 5709 3196 50  0000 L CNN
 F 1 "R_Small" H 5709 3105 50  0000 L CNN
-F 2 "" H 5650 3150 50  0001 C CNN
+F 2 "Resistor_SMD:R_0603_1608Metric" H 5650 3150 50  0001 C CNN
 F 3 "~" H 5650 3150 50  0001 C CNN
 	1    5650 3150
@@
 F 0 "R1" V 3450 4400 50  0000 C CNN
 F 1 "10k" V 3300 4300 50  0000 C CNN
-F 2 "" H 3400 4250 50  0001 C CNN
+F 2 "Resistor_SMD:R_0603_1608Metric" H 3400 4250 50  0001 C CNN
 F 3 "~" H 3400 4250 50  0001 C CNN
 	1    3400 4250
@@
 L power:VCC #PWR0109
 U 1 1 5F5FA394
-P 1950 5350
-F 0 "#PWR0109" H 1950 5200 50  0001 C CNN
-F 1 "VCC" H 1965 5523 50  0000 C CNN
-F 2 "" H 1950 5350 50  0001 C CNN
-F 3 "" H 1950 5350 50  0001 C CNN
-	1    1950 5350
+P 2800 5300
+F 0 "#PWR0109" H 2800 5150 50  0001 C CNN
+F 1 "VCC" H 2815 5473 50  0000 C CNN
+F 2 "" H 2800 5300 50  0001 C CNN
+F 3 "" H 2800 5300 50  0001 C CNN
+	1    2800 5300
 	1    0    0    -1
 $EndComp
@@
 Wire Wire Line
 	2800 5650 2600 5650
-Wire Wire Line
-	2100 5450 1950 5450
-Wire Wire Line
-	1950 5450 1950 5350
-Text Label 2850 5450 2    50   ~ 0
+Text Label 1850 5450 0    50   ~ 0
 MISO
 Text Label 2850 5550 2    50   ~ 0
@@
 RESET
 Wire Wire Line
-	2850 5450 2600 5450
-Wire Wire Line
 	2850 5550 2600 5550
 Wire Wire Line
@@
 Wire Wire Line
 	2100 5650 1850 5650
+$Comp
+L Sensor_Touch:AT42QT1010-TSHR U3
+U 1 1 5F607756
+P 7750 3600
+F 0 "U3" H 8000 3350 50  0000 C CNN
+F 1 "AT42QT1010-TSHR" H 8150 3850 50  0000 C CNN
+F 2 "Package_TO_SOT_SMD:SOT-23-6" H 7800 3350 50  0001 L CNN
+F 3 "http://ww1.microchip.com/downloads/en/DeviceDoc/40001946A.pdf" H 8020 4150 50  0001 C CNN
+	1    7750 3600
+	1    0    0    -1
+$EndComp
+Text Label 3250 4150 2    50   ~ 0
+PB2
+NoConn ~ 2950 3750
+Wire Wire Line
+	3250 4150 2950 4150
+$Comp
+L Device:C_Small C5
+U 1 1 5F611C94
+P 8450 3600
+F 0 "C5" H 8542 3646 50  0000 L CNN
+F 1 "10n" H 8542 3555 50  0000 L CNN
+F 2 "Capacitor_SMD:C_0603_1608Metric" H 8450 3600 50  0001 C CNN
+F 3 "~" H 8450 3600 50  0001 C CNN
+	1    8450 3600
+	1    0    0    -1
+$EndComp
+$Comp
+L Device:R_Small R8
+U 1 1 5F612070
+P 8950 3500
+F 0 "R8" V 8754 3500 50  0000 C CNN
+F 1 "10k" V 8845 3500 50  0000 C CNN
+F 2 "Resistor_SMD:R_0603_1608Metric" H 8950 3500 50  0001 C CNN
+F 3 "~" H 8950 3500 50  0001 C CNN
+	1    8950 3500
+	0    1    1    0
+$EndComp
+Wire Wire Line
+	8850 3500 8450 3500
+Wire Wire Line
+	8450 3500 8150 3500
+Connection ~ 8450 3500
+Wire Wire Line
+	8150 3700 8450 3700
+$Comp
+L power:GND #PWR03
+U 1 1 5F617585
+P 7750 3950
+F 0 "#PWR03" H 7750 3700 50  0001 C CNN
+F 1 "GND" H 7755 3777 50  0000 C CNN
+F 2 "" H 7750 3950 50  0001 C CNN
+F 3 "" H 7750 3950 50  0001 C CNN
+	1    7750 3950
+	1    0    0    -1
+$EndComp
+$Comp
+L power:VCC #PWR02
+U 1 1 5F617760
+P 7750 3250
+F 0 "#PWR02" H 7750 3100 50  0001 C CNN
+F 1 "VCC" H 7765 3423 50  0000 C CNN
+F 2 "" H 7750 3250 50  0001 C CNN
+F 3 "" H 7750 3250 50  0001 C CNN
+	1    7750 3250
+	1    0    0    -1
+$EndComp
+Wire Wire Line
+	7750 3250 7750 3300
+Wire Wire Line
+	7750 3900 7750 3950
+$Comp
+L power:GND #PWR01
+U 1 1 5F61B171
+P 7150 3400
+F 0 "#PWR01" H 7150 3150 50  0001 C CNN
+F 1 "GND" H 7155 3227 50  0000 C CNN
+F 2 "" H 7150 3400 50  0001 C CNN
+F 3 "" H 7150 3400 50  0001 C CNN
+	1    7150 3400
+	1    0    0    -1
+$EndComp
+Wire Wire Line
+	7150 3400 7150 3350
+Wire Wire Line
+	7150 3350 7350 3350
+Wire Wire Line
+	7350 3350 7350 3500
+Wire Wire Line
+	7350 3700 7100 3700
+Text Label 7100 3700 0    50   ~ 0
+PB2
+$Comp
+L Connector:TestPoint TP1
+U 1 1 5F6208B4
+P 9300 3500
+F 0 "TP1" H 9358 3618 50  0000 L CNN
+F 1 "Touch" H 9358 3527 50  0000 L CNN
+F 2 "" H 9500 3500 50  0001 C CNN
+F 3 "~" H 9500 3500 50  0001 C CNN
+	1    9300 3500
+	1    0    0    -1
+$EndComp
+Wire Wire Line
+	9300 3500 9050 3500
+Wire Wire Line
+	1850 5450 2100 5450
+Wire Wire Line
+	2800 5300 2800 5450
+Wire Wire Line
+	2800 5450 2600 5450
 $EndSCHEMATC

Commit message: Tape out ornament.
Parts:
- added C6: 0.1u, Capacitor_SMD:C_0603_1608Metric, symbol Device:C_Small
- C1: value C_Small -> 0.1u
- J1: footprint (none) -> Matir:AVR_ISP
- R2, R3, R4, R5, R6, R7: value R_Small -> 200
- TP1: footprint (none) -> Matir:TOUCH_SINGLE
- U2: footprint (none) -> Matir:DRV_WSON6
Connections:
- net GND: now also C6.2
- net VCC: now also C6.1
Other:
- moved on the sheet: C1
Changed lines of the file:
@@
 F 0 "U2" H 2850 2415 50  0000 C CNN
 F 1 "TPS61099X" H 2850 2324 50  0000 C CNN
-F 2 "" H 2850 1850 50  0001 C CNN
+F 2 "Matir:DRV_WSON6" H 2850 1850 50  0001 C CNN
 F 3 "" H 2850 1850 50  0001 C CNN
 	1    2850 1850
@@
 L Device:C_Small C1
 U 1 1 5F5D15F5
-P 1050 2950
-F 0 "C1" H 1142 2996 50  0000 L CNN
-F 1 "C_Small" H 1142 2905 50  0000 L CNN
-F 2 "Capacitor_SMD:C_0603_1608Metric" H 1050 2950 50  0001 C CNN
-F 3 "~" H 1050 2950 50  0001 C CNN
-	1    1050 2950
+P 1000 2850
+F 0 "C1" H 1092 2896 50  0000 L CNN
+F 1 "0.1u" H 1092 2805 50  0000 L CNN
+F 2 "Capacitor_SMD:C_0603_1608Metric" H 1000 2850 50  0001 C CNN
+F 3 "~" H 1000 2850 50  0001 C CNN
+	1    1000 2850
 	1    0    0    -1
 $EndComp
@@
 L power:VCC #PWR0105
 U 1 1 5F5D1899
-P 1050 2750
-F 0 "#PWR0105" H 1050 2600 50  0001 C CNN
-F 1 "VCC" H 1065 2923 50  0000 C CNN
-F 2 "" H 1050 2750 50  0001 C CNN
-F 3 "" H 1050 2750 50  0001 C CNN
-	1    1050 2750
+P 1000 2650
+F 0 "#PWR0105" H 1000 2500 50  0001 C CNN
+F 1 "VCC" H 1015 2823 50  0000 C CNN
+F 2 "" H 1000 2650 50  0001 C CNN
+F 3 "" H 1000 2650 50  0001 C CNN
+	1    1000 2650
 	1    0    0    -1
 $EndComp
@@
 L power:GND #PWR0106
 U 1 1 5F5D1B08
-P 1050 3150
-F 0 "#PWR0106" H 1050 2900 50  0001 C CNN
-F 1 "GND" H 1055 2977 50  0000 C CNN
-F 2 "" H 1050 3150 50  0001 C CNN
-F 3 "" H 1050 3150 50  0001 C CNN
-	1    1050 3150
-	1    0    0    -1
-$EndComp
-Wire Wire Line
-	1050 3050 1050 3150
-Wire Wire Line
-	1050 2850 1050 2750
+P 1000 3050
+F 0 "#PWR0106" H 1000 2800 50  0001 C CNN
+F 1 "GND" H 1005 2877 50  0000 C CNN
+F 2 "" H 1000 3050 50  0001 C CNN
+F 3 "" H 1000 3050 50  0001 C CNN
+	1    1000 3050
+	1    0    0    -1
+$EndComp
+Wire Wire Line
+	1000 2950 1000 3050
+Wire Wire Line
+	1000 2750 1000 2650
 Text Label 3250 3350 2    50   ~ 0
 PA3
@@
 P 4400 3150
 F 0 "R2" H 4459 3196 50  0000 L CNN
-F 1 "R_Small" H 4459 3105 50  0000 L CNN
+F 1 "200" H 4459 3105 50  0000 L CNN
 F 2 "Resistor_SMD:R_0603_1608Metric" H 4400 3150 50  0001 C CNN
 F 3 "~" H 4400 3150 50  0001 C CNN
@@
 P 4650 3150
 F 0 "R3" H 4709 3196 50  0000 L CNN
-F 1 "R_Small" H 4709 3105 50  0000 L CNN
+F 1 "200" H 4709 3105 50  0000 L CNN
 F 2 "Resistor_SMD:R_0603_1608Metric" H 4650 3150 50  0001 C CNN
 F 3 "~" H 4650 3150 50  0001 C CNN
@@
 P 4900 3150
 F 0 "R4" H 4959 3196 50  0000 L CNN
-F 1 "R_Small" H 4959 3105 50  0000 L CNN
+F 1 "200" H 4959 3105 50  0000 L CNN
 F 2 "Resistor_SMD:R_0603_1608Metric" H 4900 3150 50  0001 C CNN
 F 3 "~" H 4900 3150 50  0001 C CNN
@@
 P 5150 3150
 F 0 "R5" H 5209 3196 50  0000 L CNN
-F 1 "R_Small" H 5209 3105 50  0000 L CNN
+F 1 "200" H 5209 3105 50  0000 L CNN
 F 2 "Resistor_SMD:R_0603_1608Metric" H 5150 3150 50  0001 C CNN
 F 3 "~" H 5150 3150 50  0001 C CNN
@@
 P 5400 3150
 F 0 "R6" H 5459 3196 50  0000 L CNN
-F 1 "R_Small" H 5459 3105 50  0000 L CNN
+F 1 "200" H 5459 3105 50  0000 L CNN
 F 2 "Resistor_SMD:R_0603_1608Metric" H 5400 3150 50  0001 C CNN
 F 3 "~" H 5400 3150 50  0001 C CNN
@@
 P 5650 3150
 F 0 "R7" H 5709 3196 50  0000 L CNN
-F 1 "R_Small" H 5709 3105 50  0000 L CNN
+F 1 "200" H 5709 3105 50  0000 L CNN
 F 2 "Resistor_SMD:R_0603_1608Metric" H 5650 3150 50  0001 C CNN
 F 3 "~" H 5650 3150 50  0001 C CNN
@@
 F 0 "J1" H 2350 5867 50  0000 C CNN
 F 1 "PROG" H 2350 5776 50  0000 C CNN
-F 2 "" H 2300 5550 50  0001 C CNN
+F 2 "Matir:AVR_ISP" H 2300 5550 50  0001 C CNN
 F 3 "~" H 2300 5550 50  0001 C CNN
 	1    2300 5550
@@
 F 0 "TP1" H 9358 3618 50  0000 L CNN
 F 1 "Touch" H 9358 3527 50  0000 L CNN
-F 2 "" H 9500 3500 50  0001 C CNN
+F 2 "Matir:TOUCH_SINGLE" H 9500 3500 50  0001 C CNN
 F 3 "~" H 9500 3500 50  0001 C CNN
 	1    9300 3500
@@
 Wire Wire Line
 	2800 5450 2600 5450
+$Comp
+L Device:C_Small C6
+U 1 1 5F5F52AC
+P 7100 2750
+F 0 "C6" H 7192 2796 50  0000 L CNN
+F 1 "0.1u" H 7192 2705 50  0000 L CNN
+F 2 "Capacitor_SMD:C_0603_1608Metric" H 7100 2750 50  0001 C CNN
+F 3 "~" H 7100 2750 50  0001 C CNN
+	1    7100 2750
+	1    0    0    -1
+$EndComp
+$Comp
+L power:VCC #PWR04
+U 1 1 5F5F5884
+P 7100 2650
+F 0 "#PWR04" H 7100 2500 50  0001 C CNN
+F 1 "VCC" H 7115 2823 50  0000 C CNN
+F 2 "" H 7100 2650 50  0001 C CNN
+F 3 "" H 7100 2650 50  0001 C CNN
+	1    7100 2650
+	1    0    0    -1
+$EndComp
+$Comp
+L power:GND #PWR05
+U 1 1 5F5F5F4F
+P 7100 2850
+F 0 "#PWR05" H 7100 2600 50  0001 C CNN
+F 1 "GND" H 7105 2677 50  0000 C CNN
+F 2 "" H 7100 2850 50  0001 C CNN
+F 3 "" H 7100 2850 50  0001 C CNN
+	1    7100 2850
+	1    0    0    -1
+$EndComp
 $EndSCHEMATC

Commit message: Ornament bump
Parts:
- added JP1: Jumper_NO_Small, Jumper:SolderJumper-2_P1.3mm_Open_TrianglePad1.0x1.5mm, symbol Device:Jumper_NO_Small
Connections:
- net VCC: now also JP1.1
- net at BT1.1 (+), C2.1, L1.1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: now also JP1.2
Changed lines of the file:
@@
 	1    0    0    -1
 $EndComp
+$Comp
+L Device:Jumper_NO_Small JP1
+U 1 1 5F705426
+P 1650 1550
+F 0 "JP1" H 1650 1735 50  0000 C CNN
+F 1 "Jumper_NO_Small" H 1650 1644 50  0000 C CNN
+F 2 "Jumper:SolderJumper-2_P1.3mm_Open_TrianglePad1.0x1.5mm" H 1650 1550 50  0001 C CNN
+F 3 "~" H 1650 1550 50  0001 C CNN
+	1    1650 1550
+	1    0    0    -1
+$EndComp
+Wire Wire Line
+	1750 1550 1900 1550
+Connection ~ 1900 1550
+$Comp
+L power:VCC #PWR06
+U 1 1 5F7076A5
+P 1250 1500
+F 0 "#PWR06" H 1250 1350 50  0001 C CNN
+F 1 "VCC" H 1265 1673 50  0000 C CNN
+F 2 "" H 1250 1500 50  0001 C CNN
+F 3 "" H 1250 1500 50  0001 C CNN
+	1    1250 1500
+	1    0    0    -1
+$EndComp
+Wire Wire Line
+	1250 1500 1250 1550
+Wire Wire Line
+	1250 1550 1550 1550
 $EndSCHEMATC
