File: pcbs/powerlog/powerlog.kicad_pcb (KiCad board)
At the start: 2 copper layers, 44 parts, among them J1 Conn_01x06, J2 USB_B_Micro, J3 Conn_01x06, J4 TC2030, SW1 SW_Push, U1 AP2112K-3.3, U2 INA3221, U4 ATSAMD21E15B-M

Commit message: Edges
Parts:
- removed H1, H2, H3, H4: 3mm, MountingHole:MountingHole_3.2mm_M3
- moved J1 25.0 mm to (89.0, 55.5), turned to 270 degrees
- moved J3 25.0 mm to (126.2, 80.5), turned to 90 degrees
Connections:
- J1 pad 1: Net-(J1-Pad1) -> /INP_A
- J1 pad 2: /INP_C -> GND
- J1 pad 3: GND -> /INP_B
- J1 pad 4: /INP_B -> GND
- J1 pad 5: GND -> /INP_C
- J1 pad 6: /INP_A -> Net-(J1-Pad6)
- J3 pad 1: /OUT_A -> Net-(J1-Pad6)
- J3 pad 2: GND -> /OUT_C
- J3 pad 3: /OUT_B -> GND
- J3 pad 4: GND -> /OUT_B
- J3 pad 5: /OUT_C -> GND
- J3 pad 6: Net-(J1-Pad1) -> /OUT_A
Routing:
- net Net-(J1-Pad6): track 0.00 -> 40.0 mm
- net Net-(J1-Pad1): track 40.0 -> 0.00 mm
Other:
- board outline added: 44.2 x 49.8 mm

Commit message: Layout
Parts:
- moved C8 2.00 mm to (113.0, 99.2)
- moved R14 2.00 mm to (113.1, 97.5)
- moved R15 2.00 mm to (113.1, 95.8)
- moved J2 1.00 mm to (103.5, 98.8)
- moved R1 1.00 mm to (108.8, 98.2)
- moved SW1 0.90 mm to (120.5, 97.8)
Connections:
- J1 pad 6: Net-(J1-Pad6) -> GND
- J3 pad 1: Net-(J1-Pad6) -> GND
Routing:
- net Net-(J1-Pad6): track 40.0 -> 0.00 mm
- net GND: track 128.4 -> 167.5 mm
- net +3V3: track 90.9 -> 88.9 mm
- net /~RST: track 18.7 -> 17.3 mm
- net /USB_P: track 4.36 -> 3.36 mm
- net /USB_N: track 4.30 -> 3.30 mm
- net +5V: track 17.1 -> 18.1 mm
- net Net-(R14-Pad2): track 12.0 -> 11.4 mm
Other:
- board size 44.2 x 49.8 mm -> 44.2 x 48.8 mm
- board text added: "(C) 2021 Matir https://github.com/Matir/"
- board text added: "-"
- board text added: "All Grounds Are Common! CH1/CH2/CH3/USB"
- board text added: "CH1+"
- board text added: "CH2+"
- board text added: "CH3+"
- board text added: "Powerlog"
