File: pcbs/powerlog/powerlog.sch (KiCad schematic (older format))
At the start: 38 parts, among them J1 Conn_01x04, J2 USB_B_Micro, J3 Conn_01x04, J4 TC2030, SW1 SW_Push, U1 AP2112K-3.3, U2 INA219BxDCN, U3 INA219BxDCN, U4 ATSAMD21E15B-M

Commit message: Continue powerlog
Parts:
- removed J1, J3: Conn_01x04, symbol Connector_Generic:Conn_01x04
- removed U2, U3: INA219BxDCN, Package_TO_SOT_SMD:SOT-23-8, symbol Analog_ADC:INA219BxDCN
- added J1, J3: Conn_01x06, TerminalBlock_Phoenix:TerminalBlock_Phoenix_PT-1,5-6-5.0-H_1x06_P5.00mm_Horizontal, symbol Connector_Generic:Conn_01x06
- added R16: 25m, Resistor_SMD:R_2512_6332Metric, symbol Device:R_Small
- added R17, R18: 10, Resistor_SMD:R_0603_1608Metric, symbol Device:R_Small
- added U2: INA3221, Package_DFN_QFN:Texas_RGV_S-PVQFN-N16_EP2.1x2.1mm, symbol Power_Management:INA3221
- C2, C3: value C_Small -> 0.1u
- C4: value 0.1 -> 0.1u
- J4: footprint (none) -> Connector:Tag-Connect_TC2030-IDC-NL_2x03_P1.27mm_Vertical
- R1: value R_Small -> 0/NP
- R10, R12: value 3.3k -> 10k
- R11, R13, R8, R9: value R_Small -> 1k
- R4: value 25m -> 10; footprint Resistor_SMD:R_2512_6332Metric -> Resistor_SMD:R_0603_1608Metric
- R6: value 10 -> 25m; footprint Resistor_SMD:R_0603_1608Metric -> Resistor_SMD:R_2512_6332Metric
- SW1: footprint (none) -> Button_Switch_SMD:SW_SPST_PTS645
Connections:
- net labels added: INP_C, OUT_C
- wire segments 139 -> 157
- no-connect marks 19 -> 23
Other:
- moved on the sheet: C3, C5, R3, R5, R7

Commit message: First pass routing.
Parts:
- added H1, H2, H3, H4: 3mm, MountingHole:MountingHole_3.2mm_M3, symbol Mechanical:MountingHole
Connections:
- net INP_A: now also R5.1, R7.1; no longer R3.1, R5.2
- net INP_B: now also R17.1, R6.1; no longer R2.1, R6.2
- net INP_C: now also R16.1, R18.1; no longer R16.2, R4.1
- net LED_1: now also D2.1 (K); no longer D4.1 (K)
- net LED_3: now also D4.1 (K); no longer D2.1 (K)
- net OUT_A: now also R3.1, R5.2; no longer R5.1, R7.1
- net OUT_B: now also R2.1, R6.2; no longer R17.1, R6.1
- net OUT_C: now also R16.2, R4.1; no longer R16.1, R18.1
- net IN-1: now reaches C3.1, R3.2, U2.11 (IN-1)
- net IN+1: now reaches C3.2, R7.2, U2.12 (IN+1)
- net IN-3: now reaches C4.1, R4.2, U2.1 (IN-3)
- net IN-2: now reaches C2.1, R2.2, U2.14 (IN-2)
- net IN+2: now reaches C2.2, R17.2, U2.15 (IN+2)
- net IN+3: now reaches C4.2, R18.2, U2.2 (IN+3)
Changed lines of the file:
@@
 Connection ~ 2400 4150
 Text Label 2100 4150 0    50   ~ 0
+OUT_A
+Text Label 3100 4150 2    50   ~ 0
 INP_A
-Text Label 3100 4150 2    50   ~ 0
-OUT_A
 $Comp
 L power:GND #PWR010
@@
 	4550 3100 5500 3100
 Text Label 5500 2900 2    50   ~ 0
-LED_1
+LED_3
 Text Label 5500 3000 2    50   ~ 0
 LED_2
 Text Label 5500 3100 2    50   ~ 0
-LED_3
+LED_1
 Wire Wire Line
 	7950 1650 7650 1650
@@
 Connection ~ 1600 4450
 Text Label 1300 4450 0    50   ~ 0
+OUT_B
+Text Label 2300 4450 2    50   ~ 0
 INP_B
-Text Label 2300 4450 2    50   ~ 0
-OUT_B
 Wire Wire Line
 	1600 4800 1600 4900
@@
 Connection ~ 1600 5250
 Text Label 1300 5250 0    50   ~ 0
+OUT_C
+Text Label 2300 5250 2    50   ~ 0
 INP_C
-Text Label 2300 5250 2    50   ~ 0
-OUT_C
 Wire Wire Line
 	1600 5600 1600 5700
@@
 Text Label 1300 1250 2    50   ~ 0
 INP_C
+$Comp
+L Mechanical:MountingHole H3
+U 1 1 60464762
+P 10250 5800
+F 0 "H3" H 10350 5846 50  0000 L CNN
+F 1 "3mm" H 10350 5755 50  0000 L CNN
+F 2 "MountingHole:MountingHole_3.2mm_M3" H 10250 5800 50  0001 C CNN
+F 3 "~" H 10250 5800 50  0001 C CNN
+	1    10250 5800
+	1    0    0    -1
+$EndComp
+$Comp
+L Mechanical:MountingHole H4
+U 1 1 60464A41
+P 10250 6000
+F 0 "H4" H 10350 6046 50  0000 L CNN
+F 1 "3mm" H 10350 5955 50  0000 L CNN
+F 2 "MountingHole:MountingHole_3.2mm_M3" H 10250 6000 50  0001 C CNN
+F 3 "~" H 10250 6000 50  0001 C CNN
+	1    10250 6000
+	1    0    0    -1
+$EndComp
+$Comp
+L Mechanical:MountingHole H1
+U 1 1 60464C19
+P 10050 5800
+F 0 "H1" H 10150 5846 50  0000 L CNN
+F 1 "3mm" H 10150 5755 50  0000 L CNN
+F 2 "MountingHole:MountingHole_3.2mm_M3" H 10050 5800 50  0001 C CNN
+F 3 "~" H 10050 5800 50  0001 C CNN
+	1    10050 5800
+	1    0    0    -1
+$EndComp
+$Comp
+L Mechanical:MountingHole H2
+U 1 1 60464E90
+P 10050 6000
+F 0 "H2" H 10150 6046 50  0000 L CNN
+F 1 "3mm" H 10150 5955 50  0000 L CNN
+F 2 "MountingHole:MountingHole_3.2mm_M3" H 10050 6000 50  0001 C CNN
+F 3 "~" H 10050 6000 50  0001 C CNN
+	1    10050 6000
+	1    0    0    -1
+$EndComp
+Text Label 2850 4600 0    50   ~ 0
+IN+1
+Text Label 2850 4900 0    50   ~ 0
+IN+2
+Text Label 2850 4700 0    50   ~ 0
+IN-1
+Text Label 2850 5000 0    50   ~ 0
+IN-2
+Text Label 2850 5200 0    50   ~ 0
+IN+3
+Text Label 2850 5300 0    50   ~ 0
+IN-3
 $EndSCHEMATC

Commit message: Edges
Parts:
- removed H1, H2, H3, H4: 3mm, MountingHole:MountingHole_3.2mm_M3, symbol Mechanical:MountingHole
Connections:
- net GND: now also J1.2 (Pin_2), J1.4 (Pin_4), J3.3 (Pin_3), J3.5 (Pin_5); no longer J1.3 (Pin_3), J1.5 (Pin_5), J3.2 (Pin_2), J3.4 (Pin_4)
- net INP_A: now also J1.1 (Pin_1); no longer J1.6 (Pin_6)
- net INP_B: now also J1.3 (Pin_3); no longer J1.4 (Pin_4)
- net INP_C: now also J1.5 (Pin_5); no longer J1.2 (Pin_2)
- net OUT_A: now also J3.6 (Pin_6); no longer J3.1 (Pin_1)
- net OUT_B: now also J3.4 (Pin_4); no longer J3.3 (Pin_3)
- net OUT_C: now also J3.2 (Pin_2); no longer J3.5 (Pin_5)
- new net: J1.6 (Pin_6), J3.1 (Pin_1)
Changed lines of the file:
@@
 L Connector_Generic:Conn_01x06 J3
 U 1 1 60435955
-P 2100 1050
-F 0 "J3" H 2180 1042 50  0000 L CNN
-F 1 "Conn_01x06" H 2180 951 50  0000 L CNN
-F 2 "TerminalBlock_Phoenix:TerminalBlock_Phoenix_PT-1,5-6-5.0-H_1x06_P5.00mm_Horizontal" H 2100 1050 50  0001 C CNN
-F 3 "~" H 2100 1050 50  0001 C CNN
-	1    2100 1050
-	1    0    0    -1
-$EndComp
-$Comp
-L Connector_Generic:Conn_01x06 J1
-U 1 1 60435D1F
-P 850 1150
-F 0 "J1" H 768 625 50  0000 C CNN
-F 1 "Conn_01x06" H 768 716 50  0000 C CNN
-F 2 "TerminalBlock_Phoenix:TerminalBlock_Phoenix_PT-1,5-6-5.0-H_1x06_P5.00mm_Horizontal" H 850 1150 50  0001 C CNN
-F 3 "~" H 850 1150 50  0001 C CNN
-	1    850  1150
-	-1   0    0    1
+P 2100 1150
+F 0 "J3" H 2018 625 50  0000 C CNN
+F 1 "Conn_01x06" H 2018 716 50  0000 C CNN
+F 2 "TerminalBlock_Phoenix:TerminalBlock_Phoenix_PT-1,5-6-5.0-H_1x06_P5.00mm_Horizontal" H 2100 1150 50  0001 C CNN
+F 3 "~" H 2100 1150 50  0001 C CNN
+	1    2100 1150
+	1    0    0    1
 $EndComp
 Wire Wire Line
@@
 Text Label 1300 1250 2    50   ~ 0
 INP_C
-$Comp
-L Mechanical:MountingHole H3
-U 1 1 60464762
-P 10250 5800
-F 0 "H3" H 10350 5846 50  0000 L CNN
-F 1 "3mm" H 10350 5755 50  0000 L CNN
-F 2 "MountingHole:MountingHole_3.2mm_M3" H 10250 5800 50  0001 C CNN
-F 3 "~" H 10250 5800 50  0001 C CNN
-	1    10250 5800
-	1    0    0    -1
-$EndComp
-$Comp
-L Mechanical:MountingHole H4
-U 1 1 60464A41
-P 10250 6000
-F 0 "H4" H 10350 6046 50  0000 L CNN
-F 1 "3mm" H 10350 5955 50  0000 L CNN
-F 2 "MountingHole:MountingHole_3.2mm_M3" H 10250 6000 50  0001 C CNN
-F 3 "~" H 10250 6000 50  0001 C CNN
-	1    10250 6000
-	1    0    0    -1
-$EndComp
-$Comp
-L Mechanical:MountingHole H1
-U 1 1 60464C19
-P 10050 5800
-F 0 "H1" H 10150 5846 50  0000 L CNN
-F 1 "3mm" H 10150 5755 50  0000 L CNN
-F 2 "MountingHole:MountingHole_3.2mm_M3" H 10050 5800 50  0001 C CNN
-F 3 "~" H 10050 5800 50  0001 C CNN
-	1    10050 5800
-	1    0    0    -1
-$EndComp
-$Comp
-L Mechanical:MountingHole H2
-U 1 1 60464E90
-P 10050 6000
-F 0 "H2" H 10150 6046 50  0000 L CNN
-F 1 "3mm" H 10150 5955 50  0000 L CNN
-F 2 "MountingHole:MountingHole_3.2mm_M3" H 10050 6000 50  0001 C CNN
-F 3 "~" H 10050 6000 50  0001 C CNN
-	1    10050 6000
-	1    0    0    -1
-$EndComp
 Text Label 2850 4600 0    50   ~ 0
 IN+1
@@
 Text Label 2850 5300 0    50   ~ 0
 IN-3
+$Comp
+L Connector_Generic:Conn_01x06 J1
+U 1 1 60435D1F
+P 850 1050
+F 0 "J1" H 768 1467 50  0000 C CNN
+F 1 "Conn_01x06" H 768 1376 50  0000 C CNN
+F 2 "TerminalBlock_Phoenix:TerminalBlock_Phoenix_PT-1,5-6-5.0-H_1x06_P5.00mm_Horizontal" H 850 1050 50  0001 C CNN
+F 3 "~" H 850 1050 50  0001 C CNN
+	1    850  1050
+	-1   0    0    -1
+$EndComp
 $EndSCHEMATC

Commit message: Layout
Connections:
- net GND: now also J1.6 (Pin_6), J3.1 (Pin_1)
Changed lines of the file:
@@
 $EndComp
 Wire Wire Line
-	1050 1350 1900 1350
+	1050 1350 1450 1350
 Wire Wire Line
-	1450 1150 1450 1500
+	1450 1150 1450 1350
 Wire Wire Line
 	1050 1250 1300 1250
@@
 	-1   0    0    -1
 $EndComp
+Connection ~ 1450 1350
+Wire Wire Line
+	1450 1350 1900 1350
+Wire Wire Line
+	1450 1350 1450 1500
 $EndSCHEMATC

Commit message: Update powerlog
Parts:
- U4: symbol MCU_Microchip_SAMD:ATSAMD21E15B-M -> powerlog-rescue:ATSAMD21E15B-M-MCU_Microchip_SAMD
Changed lines of the file:
@@
 Connection ~ 3000 2150
 $Comp
-L MCU_Microchip_SAMD:ATSAMD21E15B-M U4
+L powerlog-rescue:ATSAMD21E15B-M-MCU_Microchip_SAMD U4
 U 1 1 60175019
 P 8650 3250
