File: pcbs/ledpanel/ledpanel.kicad_pcb (KiCad board)
At the start: 2 copper layers, 80 x 80 mm, 40 parts, among them J1 Male_Pins, J2 Female_Socket, J3 Screw, J4 Screw

Commit message: Finish ledpanel
Routing:
- net GND: track 0.00 -> 84.1 mm, vias 0 -> 40
- net Net-(D8-Pad1): track 0.00 -> 7.85 mm
- net Net-(D5-Pad1): track 0.00 -> 7.85 mm
- net Net-(D2-Pad1): track 0.00 -> 7.85 mm
- net Net-(D11-Pad1): track 0.00 -> 7.85 mm
- net Net-(D23-Pad1): track 0.00 -> 7.70 mm
- net Net-(D20-Pad1): track 0.00 -> 7.70 mm
- net Net-(D17-Pad1): track 0.00 -> 7.70 mm
- net Net-(D14-Pad1): track 0.00 -> 7.70 mm
- net Net-(D7-Pad1): track 0.00 -> 7.55 mm
- net Net-(D4-Pad1): track 0.00 -> 7.55 mm
- net Net-(D10-Pad1): track 0.00 -> 7.55 mm
- net Net-(D1-Pad1): track 0.00 -> 7.55 mm
- net Net-(D19-Pad1): track 0.00 -> 6.80 mm
- net Net-(D16-Pad1): track 0.00 -> 6.80 mm
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Other:
- board text added: "+"
- board text added: "-"
- board text added: "LED Panel (c) 2021 Matir"
