File: pcbs/espctl/espctl.sch (KiCad schematic (older format))
At the start: 33 parts, among them J1 Screw_Terminal_01x02, J2 Barrel_Jack_Switch, J3 Conn_01x03, J4 Screw_Terminal_01x02, J5 Screw_Terminal_01x02, J6 Screw_Terminal_01x02, J7 Conn_01x06, Q1 NX3008NBK, Q2 NX3008NBK, Q3 NX3008NBK, Q4 PMV33UPE, Q5 PMV33UPE, Q6 PMV33UPE, SW1 SW_Push, SW2 SW_Push, U1 AP2112K-3.3, U2 ESP32-WROOM-32D

Commit message: espctl layout
Parts:
- removed J7: Conn_01x06, Connector_PinHeader_2.54mm:PinHeader_2x03_P2.54mm_Vertical, symbol Connector_Generic:Conn_01x06
- TP1: footprint TestPoint:TestPoint_Loop_D1.80mm_Drill1.0mm_Beaded -> TestPoint:TestPoint_Pad_D1.0mm
Connections:
- net CH1: now also U2.12 (IO27); no longer U2.28 (IO17)
- no-connect marks 23 -> 27
Changed lines of the file:
@@
 F 0 "TP1" H 2208 1668 50  0000 L CNN
 F 1 "TP5V" H 2208 1577 50  0000 L CNN
-F 2 "TestPoint:TestPoint_Loop_D1.80mm_Drill1.0mm_Beaded" H 2350 1550 50  0001 C CNN
+F 2 "TestPoint:TestPoint_Pad_D1.0mm" H 2350 1550 50  0001 C CNN
 F 3 "~" H 2350 1550 50  0001 C CNN
 	1    2150 1550
@@
 NoConn ~ 4850 2750
 Wire Wire Line
-	6050 3550 6400 3550
+	6050 4350 6400 4350
 Wire Wire Line
 	6050 3650 6400 3650
 Wire Wire Line
 	6050 3750 6400 3750
-Text Label 6400 3550 2    50   ~ 0
+Text Label 6400 4350 2    50   ~ 0
 CH1
 Text Label 6400 3650 2    50   ~ 0
@@
 NoConn ~ 6050 4150
 NoConn ~ 6050 4250
-NoConn ~ 6050 4350
 NoConn ~ 6050 4450
 NoConn ~ 6050 4550
@@
 	1    0    0    -1
 $EndComp
-$Comp
-L Connector_Generic:Conn_01x06 J7
-U 1 1 606DC5A1
-P 3500 3900
-F 0 "J7" H 3580 3892 50  0000 L CNN
-F 1 "Conn_01x06" H 3580 3801 50  0000 L CNN
-F 2 "Connector_PinHeader_2.54mm:PinHeader_2x03_P2.54mm_Vertical" H 3500 3900 50  0001 C CNN
-F 3 "~" H 3500 3900 50  0001 C CNN
-	1    3500 3900
-	1    0    0    -1
-$EndComp
-$Comp
-L power:GND #PWR023
-U 1 1 606DD72D
-P 3100 3700
-F 0 "#PWR023" H 3100 3450 50  0001 C CNN
-F 1 "GND" V 3105 3572 50  0000 R CNN
-F 2 "" H 3100 3700 50  0001 C CNN
-F 3 "" H 3100 3700 50  0001 C CNN
-	1    3100 3700
-	0    1    1    0
-$EndComp
-Wire Wire Line
-	3100 3700 3300 3700
-Wire Wire Line
-	3300 3800 3050 3800
-Wire Wire Line
-	3300 3900 3050 3900
-Wire Wire Line
-	3300 4000 3050 4000
-Wire Wire Line
-	3300 4100 3050 4100
-Wire Wire Line
-	3300 4200 3050 4200
-Text Label 3050 3800 0    50   ~ 0
-MTDI
-Text Label 3050 3900 0    50   ~ 0
-MTCK
-Text Label 3050 4000 0    50   ~ 0
-MTMS
-Text Label 3050 4100 0    50   ~ 0
-MTDO
-Text Label 3050 4200 0    50   ~ 0
-~RST
 Text Label 4850 2450 2    50   ~ 0
 ~RST
@@
 	1    0    0    -1
 $EndComp
+NoConn ~ 6400 3050
+NoConn ~ 6400 3150
+NoConn ~ 6400 3250
+NoConn ~ 6400 3350
+NoConn ~ 6050 3550
 $EndSCHEMATC
