File: pcbs/espctl/espctl.kicad_pcb (KiCad board)
At the start: 2 copper layers, 33 parts, among them J1 Screw_Terminal_01x02, J2 Barrel_Jack_Switch, J3 Conn_01x03, J4 Screw_Terminal_01x02, J5 Screw_Terminal_01x02, J6 Screw_Terminal_01x02, J7 Conn_01x06, Q1 NX3008NBK, Q2 NX3008NBK, Q3 NX3008NBK, Q4 PMV33UPE, Q5 PMV33UPE, Q6 PMV33UPE, SW1 SW_Push, SW2 SW_Push, U1 AP2112K-3.3, U2 ESP32-WROOM-32D

Commit message: espctl layout
Parts:
- removed J7: Conn_01x06, Connector_PinHeader_2.54mm:PinHeader_2x03_P2.54mm_Vertical
- TP1: footprint TestPoint:TestPoint_Loop_D1.80mm_Drill1.0mm_Beaded -> TestPoint:TestPoint_Pad_D1.0mm
- moved SW1 28.3 mm to (37.2, 68.1), turned to 90 degrees
- moved R10 7.65 mm to (57.5, 79.4)
- moved R8 7.65 mm to (45.8, 79.4)
- moved R6 7.34 mm to (34.0, 79.4)
- moved Q4 6.78 mm to (36.6, 83.0)
- moved J4 6.74 mm to (35.4, 90.0)
- moved J5 6.74 mm to (47.3, 90.0)
- moved Q2 6.74 mm to (48.4, 79.3)
- moved Q3 6.74 mm to (60.1, 79.3)
- moved Q5 6.74 mm to (48.4, 83.1)
- moved Q6 6.74 mm to (60.1, 83.1)
- moved R7 6.74 mm to (51.0, 80.2)
- moved J6 6.74 mm to (59.2, 90.0)
- moved R5 6.74 mm to (39.2, 79.9)
- moved R9 6.74 mm to (62.7, 80.2)
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Connections:
- U2 pad 12: Net-(U2-Pad12) -> /CH1
- U2 pad 28: /CH1 -> Net-(U2-Pad28)
Routing:
- net GND: track 0.00 -> 82.8 mm, vias 0 -> 10
- net +5V: track 0.00 -> 76.8 mm
- net /CH2: track 0.00 -> 29.0 mm
- net /CH3: track 0.00 -> 19.3 mm
- net /~RST: track 0.00 -> 16.0 mm
- net +3V3: track 0.00 -> 14.8 mm
- net /CH1: track 0.00 -> 12.0 mm
- net Net-(Q1-Pad3): track 0.00 -> 9.72 mm, vias 0 -> 2
- net Net-(Q2-Pad3): track 0.00 -> 9.44 mm, vias 0 -> 2
- net Net-(SW2-Pad1): track 0.00 -> 8.11 mm
- net Net-(Q3-Pad3): track 0.00 -> 7.79 mm
- net /OUT1: track 0.00 -> 7.03 mm
- net /OUT3: track 0.00 -> 6.94 mm
- net /OUT2: track 0.00 -> 6.94 mm
- net /TXD: track 0.00 -> 4.44 mm
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- added copper zone on F.Cu, net +5V
- added copper zone on B.Cu, net GND
- added copper zone on F.Cu, net GND
Other:
- board outline added: 46 x 42 mm

Commit message: espctl v1 pcb
Parts:
- added REF**: MountingHole_3.2mm_M3, MountingHole:MountingHole_3.2mm_M3, F.Cu at (24.8, 90.0)
- renumbered SW2 to BOOT0, SW1 to RST, TP3 to TP3v3, TP1 to TP5V, TP2 to TPGND
Other:
- board text added: "+"
- board text added: "-"
- board text added: "ESP32 PWM CTL (C) 2021 Matir"
- board text added: "G TX RX"
Changed lines of the file:
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@@
   (general
     (thickness 1.6)
-    (drawings 4)
+    (drawings 14)
     (tracks 164)
     (zones 0)
-    (modules 32)
+    (modules 33)
     (nets 49)
   )
@@
     (add_net "Net-(U2-Pad9)")
   )
+  (module MountingHole:MountingHole_3.2mm_M3 (layer F.Cu)
+    (at 24.8 90)
+    (descr "Mounting Hole 3.2mm, no annular, M3")
+    (tags "mounting hole 3.2mm no annular m3")
+    (attr virtual)
+    (fp_text reference REF** (at 0 -4.2) (layer F.SilkS) hide
+      (effects (font (size 1 1) (thickness 0.15)))
+    )
+    (fp_text value MountingHole_3.2mm_M3 (at 0 4.2) (layer F.Fab)
+      (effects (font (size 1 1) (thickness 0.15)))
+    )
+    (fp_text user %R (at 0.3 0) (layer F.Fab)
+      (effects (font (size 1 1) (thickness 0.15)))
+    )
+    (fp_circle (center 0 0) (end 3.2 0) (layer Cmts.User) (width 0.15))
+    (fp_circle (center 0 0) (end 3.45 0) (layer F.CrtYd) (width 0.05))
+    (pad 1 np_thru_hole circle (at 0 0) (size 3.2 3.2) (drill 3.2) (layers *.Cu *.Mask))
+  )
   (module TestPoint:TestPoint_Pad_D1.0mm (layer F.Cu)
     (at 32.2 65.3)
@@
     (tags "test point SMD pad")
     (attr virtual)
-    (fp_text reference TP1 (at 0 -1.448) (layer F.SilkS)
+    (fp_text reference TP5V (at 0 -1.448) (layer F.SilkS)
       (effects (font (size 1 1) (thickness 0.15)))
     )
@@
     (tags "tactile switch Wurth Wuerth")
     (attr smd)
-    (fp_text reference SW2 (at 0.15 -2.6 90) (layer F.SilkS)
+    (fp_text reference BOOT0 (at 0.15 -2.6 90) (layer F.SilkS)
       (effects (font (size 1 1) (thickness 0.15)))
     )
@@
     (tags "tactile switch Wurth Wuerth")
     (attr smd)
-    (fp_text reference SW1 (at 0.15 -2.6 90) (layer F.SilkS)
+    (fp_text reference RST (at 0.15 -2.6 90) (layer F.SilkS)
       (effects (font (size 1 1) (thickness 0.15)))
     )
@@
     (descr "wire loop with bead as test point, loop diameter 1.8mm, hole diameter 1.0mm")
     (tags "test point wire loop bead")
-    (fp_text reference TP3 (at 0.7 2.5) (layer F.SilkS)
+    (fp_text reference TP3v3 (at 0.7 2.5) (layer F.SilkS)
       (effects (font (size 1 1) (thickness 0.15)))
     )
@@
     (descr "wire loop with bead as test point, loop diameter 1.8mm, hole diameter 1.0mm")
     (tags "test point wire loop bead")
-    (fp_text reference TP2 (at 0.7 2.5) (layer F.SilkS)
+    (fp_text reference TPGND (at 0.7 2.5) (layer F.SilkS)
       (effects (font (size 1 1) (thickness 0.15)))
     )
@@
     )
   )
+  (gr_text "ESP32 PWM CTL\n(C) 2021 Matir" (at 50.4 67.6) (layer B.SilkS)
+    (effects (font (size 1 1) (thickness 0.15)) (justify mirror))
+  )
+  (gr_text "G\nTX\nRX" (at 61.2 56.8) (layer F.SilkS)
+    (effects (font (size 1 1) (thickness 0.15)))
+  )
+  (gr_text - (at 64.2 84.4 180) (layer F.SilkS)
+    (effects (font (size 3 3) (thickness 0.3)))
+  )
+  (gr_text - (at 52.6 84.4 180) (layer F.SilkS)
+    (effects (font (size 3 3) (thickness 0.3)))
+  )
+  (gr_text - (at 40.6 84.4 180) (layer F.SilkS)
+    (effects (font (size 3 3) (thickness 0.3)))
+  )
+  (gr_text - (at 30.4 74.8 90) (layer F.SilkS)
+    (effects (font (size 3 3) (thickness 0.3)))
+  )
+  (gr_text + (at 57.4 84) (layer F.SilkS)
+    (effects (font (size 3 3) (thickness 0.3)))
+  )
+  (gr_text + (at 45.6 84) (layer F.SilkS)
+    (effects (font (size 3 3) (thickness 0.3)))
+  )
+  (gr_text + (at 33.8 83.8) (layer F.SilkS)
+    (effects (font (size 3 3) (thickness 0.3)))
+  )
+  (gr_text + (at 30.4 69) (layer F.SilkS)
+    (effects (font (size 3 3) (thickness 0.3)))
+  )
   (gr_line (start 21 94) (end 21 52) (layer Edge.Cuts) (width 0.05))
